File: ESP-12_WLED-Controller/ESP-12_WLED-Controller.sch (KiCad schematic (older format))
At the start: 23 parts, among them J1 Conn_01x04_Male, J2 Conn_01x04_Male, Q1 IRLML6344, Q2 IRF7410, SW1 SW_RST, U1 TS1117-3.3, U2 ESP-12E, U4 74LVC1G125

Commit message: Upgrade to V1.1
Added R9 gate resistor to PCB
Parts:
- added R9: 100R, Resistor_SMD:R_0805_2012Metric_Pad1.15x1.40mm_HandSolder, symbol Device:R
Connections:
- net RELAY: now also R9.2; no longer Q1.1 (G), R8.1
- new net: Q1.1 (G), R8.1, R9.1
Other:
- note added: "V1.1 - 12/2021 - P.Wulfert"
- note removed: "V1.01 - 11/2021 - P.Wulfert"
Changed lines of the file:
@@
 Wire Wire Line
 	6175 1900 6275 1900
-Text GLabel 7975 4200 0    50   Input ~ 0
+Text GLabel 7375 4200 0    50   Input ~ 0
 RELAY
 Wire Wire Line
@@
 CC BY-SA 4.0
 Text Notes 7025 7100 0    63   ~ 13
-V1.01 - 11/2021 - P.Wulfert
+V1.1 - 12/2021 - P.Wulfert
 Text Notes 10100 3725 0    35   ~ 0
 use here an alternative \nTHT P-MOSFET
@@
 Text Notes 4700 6825 0    39   ~ 0
 Use Transil-Diode as MOSFET Flyback protection.\n
+$Comp
+L Device:R R9
+U 1 1 61B66D02
+P 7825 4200
+F 0 "R9" V 7750 4175 50  0000 L CNN
+F 1 "100R" V 7825 4100 50  0000 L CNN
+F 2 "Resistor_SMD:R_0805_2012Metric_Pad1.15x1.40mm_HandSolder" V 7755 4200 50  0001 C CNN
+F 3 "~" H 7825 4200 50  0001 C CNN
+	1    7825 4200
+	0    1    1    0
+$EndComp
+Wire Wire Line
+	7375 4200 7675 4200
 $EndSCHEMATC
