File: ESP-12_WLED-Controller_KiCad6/ESP-12_WLED-Controller.kicad_pcb (KiCad board)
At the start: 2 copper layers, 58.7 x 31 mm, 29 parts, among them J1 Conn_01x04_Male, J2 Conn_01x04_Male, Q1 IRLML6344, Q2 IRF7410, SW1 SW_RST, U1 TS1117-3.3, U2 ESP-12E, U4 74LVC1G125

Commit message: Update to V2.0
Parts:
- added JP2: Jumper_2_Open, Jumper:SolderJumper-2_P1.3mm_Open_TrianglePad1.0x1.5mm, B.Cu at (165.8, 89.5)
- added aC2: 100µF, Capacitor_SMD:C_0805_2012Metric_Pad1.18x1.45mm_HandSolder, F.Cu at (120.9, 94.4)
- C1, C2: value 10nF -> 10µF
- J2: value Conn_01x04_Male -> Conn_01x05_Male; footprint Connector_PinHeader_2.54mm:PinHeader_1x04_P2.54mm_Vertical -> Connector_PinHeader_2.54mm:PinHeader_1x05_P2.54mm_Vertical
- R9: value 100R -> 300R
- moved JP1 1.03 mm to (122.6, 106.5)
- moved J2 0.34 mm to (128.5, 104.0)
- turned C2 to -90 degrees
Connections:
- net Net-(J1-Pad3) renamed DATA
- U2 pad 10: Net-(U2-Pad10) -> unconnected-(U2-Pad10)
- U2 pad 11: Net-(U2-Pad11) -> unconnected-(U2-Pad11)
- U2 pad 12: Net-(U2-Pad12) -> unconnected-(U2-Pad12)
- U2 pad 13: Net-(U2-Pad13) -> unconnected-(U2-Pad13)
- U2 pad 14: Net-(U2-Pad14) -> unconnected-(U2-Pad14)
- U2 pad 2: Net-(U2-Pad2) -> A0
- U2 pad 20: Net-(U2-Pad20) -> unconnected-(U2-Pad20)
- U2 pad 4: Net-(U2-Pad4) -> unconnected-(U2-Pad4)
- U2 pad 5: Net-(U2-Pad5) -> unconnected-(U2-Pad5)
- U2 pad 7: Net-(U2-Pad7) -> unconnected-(U2-Pad7)
- U2 pad 9: Net-(U2-Pad9) -> unconnected-(U2-Pad9)
Routing:
- net A0: track 0.00 -> 24.1 mm, vias 0 -> 1
- net DATA: track 35.2 -> 22.4 mm, vias 0 -> 1
- net GND: track 18.8 -> 31.2 mm
- net +3V3: track 82.6 -> 93.2 mm
- net +5V: track 124.3 -> 131.9 mm
- net GPIO4_5: track 3.93 -> 7.36 mm, vias 0 -> 1
- net GPIO4_3.3: track 21.5 -> 24.3 mm
- net /Reset: track 18.0 -> 15.3 mm
- net RELAY: track 24.2 -> 25.4 mm
- net WS-Strip_VCC: track 46.6 -> 47.4 mm
- net /GPIO0: track 40.0 -> 40.8 mm
Other:
- board text added: "= solder Pin"
- board text added: "A0 3V3 RX TX GND"
- board text added: "Every machine is a smoke machine if you use it wrong enough!"
- board text added: "GND TX RX 3V3 A0"
- board text added: "V2.0 - 01/2022 - P.Wulfert"
- board text removed: "3V3 RX TX GND"
- board text removed: "GND TX RX 3V3"
- board text removed: "V1.1 - 12/2021 - P.Wulfert"

Commit message: Update to V1.3
Parts:
- removed the REF** at (121.8, 89.9)
- removed the REF** at (175.4, 115.9)
- removed altQ2: alt. MOSFET, Package_TO_SOT_THT:TO-220-3_Vertical
- added C5: 100nF, Capacitor_SMD:C_0805_2012Metric_Pad1.18x1.45mm_HandSolder, F.Cu at (159.3, 89.7)
- added G***: LOGO, LOGO, B.Cu at (165.5, 97.8)
- added G***: LOGO, LOGO, B.Cu at (128.2, 91.6)
- C1, C3: footprint Capacitor_SMD:C_0805_2012Metric_Pad1.15x1.40mm_HandSolder -> Capacitor_SMD:C_0805_2012Metric_Pad1.18x1.45mm_HandSolder
- C2: value 10µF -> 47F; footprint Capacitor_SMD:C_0805_2012Metric_Pad1.15x1.40mm_HandSolder -> Capacitor_SMD:C_0805_2012Metric_Pad1.18x1.45mm_HandSolder
- J1: value Conn_01x04_Male -> Screw_Terminal_01x05; footprint TerminalBlock_Phoenix:TerminalBlock_Phoenix_MKDS-1,5-4-5.08_1x04_P5.08mm_Horizontal -> TerminalBlock:TerminalBlock_bornier-5_P5.08mm
- J2: value Conn_01x05_Male -> Conn_01x04_Male; footprint Connector_PinHeader_2.54mm:PinHeader_1x05_P2.54mm_Vertical -> Connector_PinSocket_2.54mm:PinSocket_1x04_P2.54mm_Vertical
- JP1: value Jumper -> BTN/FLASH
- JP2: footprint Jumper:SolderJumper-2_P1.3mm_Open_TrianglePad1.0x1.5mm -> Jumper:SolderJumper-2_P1.3mm_Open_RoundedPad1.0x1.5mm
- R1, R2, R3, R4, R5, R6, R7, R8, R9: footprint Resistor_SMD:R_0805_2012Metric_Pad1.15x1.40mm_HandSolder -> Resistor_SMD:R_0805_2012Metric_Pad1.20x1.40mm_HandSolder
- U4: footprint Package_SO:TSOP-5_1.65x3.05mm_P0.95mm -> Package_TO_SOT_SMD:SOT-23-5
- aC2: footprint Capacitor_SMD:C_0805_2012Metric_Pad1.18x1.45mm_HandSolder -> Capacitor_SMD:C_1206_3216Metric_Pad1.33x1.80mm_HandSolder
- moved SW1 13.7 mm to (125.8, 102.5)
- moved R7 12.2 mm to (158.8, 106.2), turned to 90 degrees
- moved C1 6.58 mm to (132.5, 92.7)
- moved C2 6.40 mm to (121.4, 92.7), turned to 90 degrees
- moved J1 4.98 mm to (173.6, 115.5)
- moved U1 4.05 mm to (127.0, 92.7)
- moved U4 3.76 mm to (159.5, 94.0)
- moved C4 3.55 mm to (160.1, 113.3), turned to 0 degrees
- moved aC2 3.45 mm to (121.4, 97.8)
- moved JP2 3.41 mm to (169.2, 89.7)
- moved R6 3.41 mm to (169.2, 89.7)
- moved J2 2.55 mm to (128.2, 106.5)
- moved Q2 2.50 mm to (164.1, 104.8), turned to 90 degrees
- moved Q1 2.04 mm to (159.4, 99.6)
- moved G*** 1.74 mm to (148.9, 106.8)
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Connections:
- net GPIO4_5 renamed DATA_5
- J1 pad 1: WS-Strip_VCC -> GND
- J1 pad 3: DATA -> WS-Strip_VCC
- J1 pad 4: GND -> DATA
- Q1 pad 3: Net-(Q1-Pad3) -> OE
- Q2 pad 4: Net-(Q1-Pad3) -> OE
- R3 pad 2: GPIO2 -> DATA_3.3
- R7 pad 2: Net-(Q1-Pad3) -> OE
- U2 pad 17: GPIO2 -> DATA_3.3
- U2 pad 19: GPIO4_3.3 -> unconnected-(U2-Pad19)
- U4 pad 1: GND -> OE
- U4 pad 2: GPIO4_3.3 -> DATA_3.3
Routing:
- net GND: track 31.2 -> 0.05 mm, vias 10 -> 1
- net +5V: track 131.9 -> 102.1 mm, vias 4 -> 10
- net WS-Strip_VCC: track 47.4 -> 21.7 mm, vias 4 -> 7
- net GPIO4_3.3: track 24.3 -> 0.00 mm, vias 2 -> 0
- net A0: track 24.1 -> 0.00 mm, vias 1 -> 0
- net OE: track 0.00 -> 20.6 mm
- net DATA_3.3: track 0.00 -> 14.9 mm, vias 0 -> 2
- net Net-(Q1-Pad3): track 12.5 -> 0.00 mm
- net +3V3: track 93.2 -> 85.7 mm
- net /GPIO0: track 40.8 -> 47.5 mm
- net DATA: track 22.4 -> 17.0 mm
- net DATA_5: track 7.36 -> 11.6 mm
- net /Reset: track 15.3 -> 11.1 mm
- net GPIO2: track 3.83 -> 0.00 mm
- net TX: track 28.1 -> 29.4 mm
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- added copper zone on B.Cu, net +5V
- added copper zone on F.Cu, net +5V
- added copper zone on F.Cu, net GND
- added copper zone on B.Cu, net WS-Strip_VCC
- added copper zone on F.Cu, net WS-Strip_VCC
Other:
- board text added: "3V3 RX TX GND"
- board text added: "GND 5V SW_5V DATA GND"
- board text added: "GND TX RX 3V3"
- board text added: "JLCJLCJLCJLC"
- board text added: "OPEN HARDWARE"
- board text added: "Thanks to WLED Project: https://github.com/Aircoookie/WLED"
- board text added: "V1.3 - 01/2022 - P.Wulfert"
- board text removed: "A0 3V3 RX TX GND"
- board text removed: "Every machine is a smoke machine if you use it wrong enough!"
- board text removed: "GND DATA 5V SW_5V"
- board text removed: "GND TX RX 3V3 A0"
- board text removed: "SW_5V 5V DATA GND"
- board text removed: "V2.0 - 01/2022 - P.Wulfert"
